File: Pi5_PCIe.kicad_pcb (KiCad board)
At the start: 4 copper layers, 50 x 50 mm, 54 parts, among them J1 12V IN, J2 Pi5 PCIe, J3 10018783-11200TLF, Q1 BS170F, U1 Mini360

Commit message: Created Gerbers for board v0.99 & tagged
Other:
- board text added: "George Smart M1GEO https://github.com/m1geo/Pi5_PCIe https://www.george-smart.co.uk Ver 0.99 - 15 Nov 2023"
- board text added: "V0.99 15/11/2023 George M1GEO"
- board text removed: "George Smart M1GEO https://github.com/m1geo/Pi5_PCIe https://www.george-smart.co.uk Ver 0.4 - 11 Nov 2023"
- board text removed: "V0.4 11/11/2023 George M1GEO"
Changed lines of the file:
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@@
       (drillshape 0)
       (scaleselection 1)
-      (outputdirectory "Gerbers/")
+      (outputdirectory "Gerbers_PCIe_V099/")
     )
   )
@@
   (gr_line (start 125 121) (end 125 79)
     (stroke (width 0.1) (type default)) (layer "Edge.Cuts"))
-  (gr_text "George Smart M1GEO\nhttps://github.com/m1geo/Pi5_PCIe\nhttps://www.george-smart.co.uk\nVer 0.4  -  11 Nov 2023" (at 157 96.5) (layer "B.SilkS")
+  (gr_text "George Smart M1GEO\nhttps://github.com/m1geo/Pi5_PCIe\nhttps://www.george-smart.co.uk\nVer 0.99  -  15 Nov 2023" (at 157 96.5) (layer "B.SilkS")
     (effects (font (size 1 1) (thickness 0.15)) (justify left bottom mirror))
   )
@@
     (effects (font (size 1 1) (thickness 0.15)) (justify left bottom))
   )
-  (gr_text "V0.4 \n11/11/2023\nGeorge M1GEO" (at 174.5 113 90) (layer "F.SilkS")
+  (gr_text "V0.99 \n15/11/2023\nGeorge M1GEO" (at 174.5 113 90) (layer "F.SilkS")
     (effects (font (size 1 1) (thickness 0.15)) (justify bottom))
   )
